File: scratchpad/QFN triple breakout/QFN triple breakout.brd (EAGLE design)
At the start: 24.1 x 14 mm, 5 parts, among them P1 SIA929DJ

Commit message: Changed a couple of part numbers to make more sense.
Parts:
- moved N1 7.62 mm to (12.7, 7.62)
- moved N2 7.62 mm to (20.3, 7.62)
Connections:
- net ND1: now also N2.D2, N2.D2$2; no longer N1.D2, N1.D2$2
- net ND2: now also N2.D1, N2.D1$1; no longer N1.D1, N1.D1$1
- net ND3: now also N1.D1, N1.D1$1; no longer N2.D1, N2.D1$1
- net ND4: now also N1.D2, N1.D2$2; no longer N2.D2, N2.D2$2
- net NG1: now also N2.G2; no longer N1.G2
- net NG2: now also N2.G1; no longer N1.G1
- net NG3: now also N1.G1; no longer N2.G1
- net NG4: now also N1.G2; no longer N2.G2
- net NS1: now also N2.S2; no longer N1.S2
- net NS2: now also N2.S1; no longer N1.S1
- net NS3: now also N1.S1; no longer N2.S1
- net NS4: now also N1.S2; no longer N2.S2
Changed lines of the file:
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@@
 <elements>
 <element name="P1" library="Railstars" package="SC70-6L" value="SIA929DJ" x="5.08" y="7.62"/>
-<element name="N2" library="Railstars" package="UDFN6" value="SSM6N55NU" x="12.7" y="7.62"/>
-<element name="N1" library="Railstars" package="UDFN6" value="SSM6N55NU" x="20.32" y="7.62"/>
+<element name="N1" library="Railstars" package="UDFN6" value="SSM6N55NU" x="12.7" y="7.62"/>
+<element name="N2" library="Railstars" package="UDFN6" value="SSM6N55NU" x="20.32" y="7.62"/>
 <element name="JP1" library="SparkFun-Connectors" package="1X09" value="M09" x="2.54" y="2.54" smashed="yes"/>
 <element name="JP2" library="SparkFun-Connectors" package="1X09" value="M09" x="2.54" y="12.7" smashed="yes"/>
@@
 <signals>
 <signal name="NG1">
-<contactref element="N1" pad="G2"/>
+<contactref element="N2" pad="G2"/>
 <contactref element="JP2" pad="8"/>
 <wire x1="20.32" y1="8.545" x2="20.32" y2="12.7" width="0.3048" layer="1"/>
 </signal>
 <signal name="NG2">
-<contactref element="N1" pad="G1"/>
+<contactref element="N2" pad="G1"/>
 <contactref element="JP1" pad="8"/>
 <wire x1="20.32" y1="6.695" x2="20.32" y2="2.54" width="0.3048" layer="1"/>
 </signal>
 <signal name="NG3">
-<contactref element="N2" pad="G1"/>
+<contactref element="N1" pad="G1"/>
 <contactref element="JP1" pad="5"/>
 <wire x1="12.7" y1="6.695" x2="12.7" y2="2.54" width="0.3048" layer="1"/>
 </signal>
 <signal name="NG4">
-<contactref element="N2" pad="G2"/>
+<contactref element="N1" pad="G2"/>
 <contactref element="JP2" pad="5"/>
 <wire x1="12.7" y1="8.545" x2="12.7" y2="12.7" width="0.3048" layer="1"/>
@@
 </signal>
 <signal name="ND2">
-<contactref element="N1" pad="D1$1"/>
-<contactref element="N1" pad="D1"/>
+<contactref element="N2" pad="D1$1"/>
+<contactref element="N2" pad="D1"/>
 <contactref element="JP2" pad="7"/>
 <wire x1="19.67" y1="8.545" x2="19.67" y2="7.795" width="0.3048" layer="1"/>
@@
 </signal>
 <signal name="NS2">
-<contactref element="N1" pad="S1"/>
+<contactref element="N2" pad="S1"/>
 <contactref element="JP1" pad="7"/>
 <wire x1="19.67" y1="6.695" x2="19.67" y2="4.43" width="0.3048" layer="1"/>
@@
 </signal>
 <signal name="NS1">
-<contactref element="N1" pad="S2"/>
+<contactref element="N2" pad="S2"/>
 <contactref element="JP2" pad="9"/>
 <wire x1="20.97" y1="8.545" x2="20.97" y2="10.81" width="0.3048" layer="1"/>
@@
 </signal>
 <signal name="ND1">
-<contactref element="N1" pad="D2"/>
-<contactref element="N1" pad="D2$2"/>
+<contactref element="N2" pad="D2"/>
+<contactref element="N2" pad="D2$2"/>
 <wire x1="20.97" y1="6.695" x2="20.97" y2="7.445" width="0.3048" layer="1"/>
 <wire x1="20.97" y1="7.445" x2="20.795" y2="7.62" width="0.3048" layer="1"/>
@@
 </signal>
 <signal name="ND3">
-<contactref element="N2" pad="D1$1"/>
-<contactref element="N2" pad="D1"/>
+<contactref element="N1" pad="D1$1"/>
+<contactref element="N1" pad="D1"/>
 <contactref element="JP2" pad="4"/>
 <wire x1="12.05" y1="8.545" x2="12.05" y2="7.795" width="0.3048" layer="1"/>
@@
 </signal>
 <signal name="NS3">
-<contactref element="N2" pad="S1"/>
+<contactref element="N1" pad="S1"/>
 <contactref element="JP1" pad="4"/>
 <wire x1="12.05" y1="6.695" x2="12.05" y2="4.43" width="0.3048" layer="1"/>
@@
 </signal>
 <signal name="NS4">
-<contactref element="N2" pad="S2"/>
+<contactref element="N1" pad="S2"/>
 <contactref element="JP2" pad="6"/>
 <wire x1="13.35" y1="8.545" x2="13.35" y2="10.81" width="0.3048" layer="1"/>
@@
 </signal>
 <signal name="ND4">
-<contactref element="N2" pad="D2"/>
-<contactref element="N2" pad="D2$2"/>
+<contactref element="N1" pad="D2"/>
+<contactref element="N1" pad="D2$2"/>
 <wire x1="13.35" y1="6.695" x2="13.35" y2="7.445" width="0.3048" layer="1"/>
 <wire x1="13.35" y1="7.445" x2="13.175" y2="7.62" width="0.3048" layer="1"/>
