File: hardware/Aegaeon REV B 20130130 PROTO.sch (EAGLE design)
At the start: 39 parts, among them IC1 ATTINY84A-MMH, Q1 DMN65D8LDW, U1 V_REG_LDOSMD

Commit message: Saved files.
Connections:
- net FORWARD: now also U$4G$1.G, U$9G$1.S; no longer U$4G$2.G, U$9G$2.S
- net REVERSE: now also U$4G$2.G, U$9G$2.S; no longer U$4G$1.G, U$9G$1.S
Changed lines of the file:
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@@
+</segment>
+<segment>
+<wire x1="45.72" y1="58.42" x2="17.78" y2="58.42" width="0.1524" layer="91"/>
+<label x="17.78" y="58.42" size="1.778" layer="95"/>
+<pinref part="U$9" gate="G$2" pin="S"/>
+<pinref part="U$4" gate="G$2" pin="G"/>
+<wire x1="45.72" y1="58.42" x2="76.2" y2="58.42" width="0.1524" layer="91"/>
+</segment>
+</net>
+<net name="FORWARD" class="0">
+<segment>
+<pinref part="IC1" gate="G$1" pin="PA7/OC0B"/>
+<wire x1="104.14" y1="160.02" x2="116.84" y2="160.02" width="0.1524" layer="91"/>
+<label x="109.22" y="160.02" size="1.778" layer="95"/>
 </segment>
 <segment>
@@
 </segment>
 </net>
-<net name="FORWARD" class="0">
-<segment>
-<pinref part="IC1" gate="G$1" pin="PA7/OC0B"/>
-<wire x1="104.14" y1="160.02" x2="116.84" y2="160.02" width="0.1524" layer="91"/>
-<label x="109.22" y="160.02" size="1.778" layer="95"/>
-</segment>
-<segment>
-<wire x1="45.72" y1="58.42" x2="17.78" y2="58.42" width="0.1524" layer="91"/>
-<label x="17.78" y="58.42" size="1.778" layer="95"/>
-<pinref part="U$9" gate="G$2" pin="S"/>
-<pinref part="U$4" gate="G$2" pin="G"/>
-<wire x1="45.72" y1="58.42" x2="76.2" y2="58.42" width="0.1524" layer="91"/>
-</segment>
-</net>
