File: hardware/Aegaeon REV C PROTO.brd (EAGLE design)
At the start: 9.2 x 16 mm, 39 parts, among them IC1 ATTINY84A-MMH, Q1 DMN65D8LDW, U1 V_REG_LDOSMD

Commit message: Feels like we're headed down a rabbit hole.
Parts:
- moved R6 5.00 mm to (6.00, 14.4), turned to 0 degrees
- moved R7 4.48 mm to (6.10, 13.4), turned to 180 degrees
- moved R11 1.30 mm to (1.35, 9.47), turned to 0 degrees
- moved R10 0.95 mm to (2.48, 9.47), turned to 180 degrees
- moved U1 0.50 mm to (7.40, 6.90)
Routing:
- net MOTOR_L: track 3.06 -> 13.9 mm, vias 1 -> 2
- net MOTOR_R: track 3.06 -> 12.7 mm, vias 1 -> 2
- net REVERSE: track 3.09 -> 8.54 mm, vias 1 -> 2
- net REV_PWM: track 1.08 -> 5.89 mm, vias 1 -> 2
- net N$11: track 0.00 -> 4.74 mm, vias 0 -> 1
- net N$1: track 4.43 -> 8.68 mm
- net FWD_PWM: track 1.46 -> 5.55 mm, vias 1 -> 2
- net N$2: track 11.0 -> 6.98 mm, vias 2 -> 0
- net GND: track 4.48 -> 8.13 mm
- net BEMF: track 14.2 -> 11.5 mm
- net 5V: track 13.3 -> 14.2 mm
- net VDCC: track 4.50 -> 3.95 mm
- net DCC_L_LL: track 18.6 -> 18.5 mm, vias 1 -> 2
